File: kicad/small_led_board/small_led_board.kicad_pcb (KiCad board)
At the start: 2 copper layers, 0 parts

Commit message: small_led_board: PCB started
Parts:
- added D1: LED, LED_THT:LED_D5.0mm, F.Cu at (71.1, 44.5)
- added D10: LED, LED_THT:LED_D5.0mm, F.Cu at (78.1, 51.4)
- added D11: LED, LED_THT:LED_D5.0mm, F.Cu at (85.1, 51.4)
- added D12: LED, LED_THT:LED_D5.0mm, F.Cu at (92.1, 51.4)
- added D13: LED, LED_THT:LED_D5.0mm, F.Cu at (99.1, 51.4)
- added D14: LED, LED_THT:LED_D5.0mm, F.Cu at (106.0, 51.4)
- added D15: LED, LED_THT:LED_D5.0mm, F.Cu at (113.0, 51.4)
- added D16: LED, LED_THT:LED_D5.0mm, F.Cu at (120.0, 51.4)
- added D17: LED, LED_THT:LED_D5.0mm, F.Cu at (71.1, 58.4)
- added D18: LED, LED_THT:LED_D5.0mm, F.Cu at (78.1, 58.4)
- added D19: LED, LED_THT:LED_D5.0mm, F.Cu at (85.1, 58.4)
- added D2: LED, LED_THT:LED_D5.0mm, F.Cu at (78.1, 44.5)
- added D20: LED, LED_THT:LED_D5.0mm, F.Cu at (92.1, 58.4)
- added D21: LED, LED_THT:LED_D5.0mm, F.Cu at (99.1, 58.4)
- added D22: LED, LED_THT:LED_D5.0mm, F.Cu at (106.0, 58.4)
- added D23: LED, LED_THT:LED_D5.0mm, F.Cu at (113.0, 58.4)
- added D24: LED, LED_THT:LED_D5.0mm, F.Cu at (120.0, 58.4)
- added D25: LED, LED_THT:LED_D5.0mm, F.Cu at (71.1, 65.4)
- added D26: LED, LED_THT:LED_D5.0mm, F.Cu at (78.1, 65.4)
- added D27: LED, LED_THT:LED_D5.0mm, F.Cu at (85.1, 65.4)
- added D28: LED, LED_THT:LED_D5.0mm, F.Cu at (92.1, 65.4)
- added D29: LED, LED_THT:LED_D5.0mm, F.Cu at (99.1, 65.4)
- added D3: LED, LED_THT:LED_D5.0mm, F.Cu at (85.1, 44.5)
- added D30: LED, LED_THT:LED_D5.0mm, F.Cu at (106.0, 65.4)
- added D31: LED, LED_THT:LED_D5.0mm, F.Cu at (113.0, 65.4)
- added D32: LED, LED_THT:LED_D5.0mm, F.Cu at (120.0, 65.4)
- added D33: LED, LED_THT:LED_D5.0mm, F.Cu at (71.1, 72.4)
- added D34: LED, LED_THT:LED_D5.0mm, F.Cu at (78.1, 72.4)
- added D35: LED, LED_THT:LED_D5.0mm, F.Cu at (85.1, 72.4)
- added D36: LED, LED_THT:LED_D5.0mm, F.Cu at (92.1, 72.4)
- added D37: LED, LED_THT:LED_D5.0mm, F.Cu at (99.1, 72.4)
- added D38: LED, LED_THT:LED_D5.0mm, F.Cu at (106.0, 72.4)
- added D39: LED, LED_THT:LED_D5.0mm, F.Cu at (113.0, 72.4)
- added D4: LED, LED_THT:LED_D5.0mm, F.Cu at (92.1, 44.5)
- added D40: LED, LED_THT:LED_D5.0mm, F.Cu at (120.0, 72.4)
- added D41: LED, LED_THT:LED_D5.0mm, F.Cu at (71.1, 79.4)
- added D42: LED, LED_THT:LED_D5.0mm, F.Cu at (78.1, 79.4)
- added D43: LED, LED_THT:LED_D5.0mm, F.Cu at (85.1, 79.4)
- added D44: LED, LED_THT:LED_D5.0mm, F.Cu at (92.1, 79.4)
- added D45: LED, LED_THT:LED_D5.0mm, F.Cu at (99.1, 79.4)
- added D46: LED, LED_THT:LED_D5.0mm, F.Cu at (106.0, 79.4)
- added D47: LED, LED_THT:LED_D5.0mm, F.Cu at (113.0, 79.4)
- added D48: LED, LED_THT:LED_D5.0mm, F.Cu at (120.0, 79.4)
- added D5: LED, LED_THT:LED_D5.0mm, F.Cu at (99.1, 44.5)
- added D6: LED, LED_THT:LED_D5.0mm, F.Cu at (106.0, 44.5)
- added D7: LED, LED_THT:LED_D5.0mm, F.Cu at (113.0, 44.5)
- added D8: LED, LED_THT:LED_D5.0mm, F.Cu at (120.0, 44.5)
- added D9: LED, LED_THT:LED_D5.0mm, F.Cu at (71.1, 51.4)
- added J1: Breakout to FPGA, Connector_PinHeader_2.54mm:PinHeader_2x06_P2.54mm_Horizontal, F.Cu at (195.6, 121.9)
- added J2: +5V IN, Connector_BarrelJack:BarrelJack_Horizontal, F.Cu at (190.0, 111.8)
- added Q1: IRLZ44N, Package_TO_SOT_THT:TO-220-3_Vertical, F.Cu at (71.1, 105.4)
- added Q10: IRF4905, Package_TO_SOT_THT:TO-220-3_Vertical, F.Cu at (127.0, 51.4)
- added Q11: IRF4905, Package_TO_SOT_THT:TO-220-3_Vertical, F.Cu at (127.0, 58.4)
- added Q12: IRF4905, Package_TO_SOT_THT:TO-220-3_Vertical, F.Cu at (127.0, 65.4)
- added Q13: IRF4905, Package_TO_SOT_THT:TO-220-3_Vertical, F.Cu at (127.0, 72.4)
- added Q14: IRF4905, Package_TO_SOT_THT:TO-220-3_Vertical, F.Cu at (127.0, 79.4)
- added Q15: IRLZ44N, Package_TO_SOT_THT:TO-220-3_Vertical, F.Cu at (137.8, 107.3)
- added Q16: IRLZ44N, Package_TO_SOT_THT:TO-220-3_Vertical, F.Cu at (137.2, 120.0)
- added Q17: IRLZ44N, Package_TO_SOT_THT:TO-220-3_Vertical, F.Cu at (137.2, 131.4)
- added Q18: IRLZ44N, Package_TO_SOT_THT:TO-220-3_Vertical, F.Cu at (177.8, 58.4)
- added Q19: IRLZ44N, Package_TO_SOT_THT:TO-220-3_Vertical, F.Cu at (177.8, 88.9)
- added Q2: IRLZ44N, Package_TO_SOT_THT:TO-220-3_Vertical, F.Cu at (78.1, 105.4)
- added Q20: IRLZ44N, Package_TO_SOT_THT:TO-220-3_Vertical, F.Cu at (177.8, 73.7)
- added Q3: IRLZ44N, Package_TO_SOT_THT:TO-220-3_Vertical, F.Cu at (85.1, 105.4)
- added Q4: IRLZ44N, Package_TO_SOT_THT:TO-220-3_Vertical, F.Cu at (92.1, 105.4)
- added Q5: IRLZ44N, Package_TO_SOT_THT:TO-220-3_Vertical, F.Cu at (99.1, 105.4)
- added Q6: IRLZ44N, Package_TO_SOT_THT:TO-220-3_Vertical, F.Cu at (106.0, 105.4)
- added Q7: IRLZ44N, Package_TO_SOT_THT:TO-220-3_Vertical, F.Cu at (113.0, 105.4)
- added Q8: IRLZ44N, Package_TO_SOT_THT:TO-220-3_Vertical, F.Cu at (120.0, 105.4)
- added Q9: IRF4905, Package_TO_SOT_THT:TO-220-3_Vertical, F.Cu at (127.0, 44.5)
- added R1: 66R, Resistor_THT:R_Axial_DIN0207_L6.3mm_D2.5mm_P7.62mm_Horizontal, F.Cu at (71.1, 94.0)
- added R10: 1K, Resistor_THT:R_Axial_DIN0207_L6.3mm_D2.5mm_P7.62mm_Horizontal, F.Cu at (71.1, 118.1)
- added R11: 1K, Resistor_THT:R_Axial_DIN0207_L6.3mm_D2.5mm_P7.62mm_Horizontal, F.Cu at (78.1, 118.1)
- added R12: 1K, Resistor_THT:R_Axial_DIN0207_L6.3mm_D2.5mm_P7.62mm_Horizontal, F.Cu at (85.1, 118.1)
- added R13: 1K, Resistor_THT:R_Axial_DIN0207_L6.3mm_D2.5mm_P7.62mm_Horizontal, F.Cu at (92.1, 118.1)
- added R14: 1K, Resistor_THT:R_Axial_DIN0207_L6.3mm_D2.5mm_P7.62mm_Horizontal, F.Cu at (99.1, 118.1)
- added R15: 1K, Resistor_THT:R_Axial_DIN0207_L6.3mm_D2.5mm_P7.62mm_Horizontal, F.Cu at (106.0, 118.1)
- added R16: 1K, Resistor_THT:R_Axial_DIN0207_L6.3mm_D2.5mm_P7.62mm_Horizontal, F.Cu at (113.0, 118.1)
- added R17: 1K, Resistor_THT:R_Axial_DIN0207_L6.3mm_D2.5mm_P7.62mm_Horizontal, F.Cu at (137.2, 44.5)
- added R18: 1K, Resistor_THT:R_Axial_DIN0207_L6.3mm_D2.5mm_P7.62mm_Horizontal, F.Cu at (137.2, 51.4)
- added R19: 1K, Resistor_THT:R_Axial_DIN0207_L6.3mm_D2.5mm_P7.62mm_Horizontal, F.Cu at (137.2, 58.4)
- added R2: 66R, Resistor_THT:R_Axial_DIN0207_L6.3mm_D2.5mm_P7.62mm_Horizontal, F.Cu at (78.1, 94.0)
- added R20: 1K, Resistor_THT:R_Axial_DIN0207_L6.3mm_D2.5mm_P7.62mm_Horizontal, F.Cu at (137.2, 65.4)
- added R21: 1K, Resistor_THT:R_Axial_DIN0207_L6.3mm_D2.5mm_P7.62mm_Horizontal, F.Cu at (137.2, 72.4)
- added R22: 1K, Resistor_THT:R_Axial_DIN0207_L6.3mm_D2.5mm_P7.62mm_Horizontal, F.Cu at (137.2, 79.4)
- added R23: 10K, Resistor_THT:R_Axial_DIN0207_L6.3mm_D2.5mm_P7.62mm_Horizontal, F.Cu at (144.8, 105.7)
- added R24: 10K, Resistor_THT:R_Axial_DIN0207_L6.3mm_D2.5mm_P7.62mm_Horizontal, F.Cu at (144.8, 118.7)
- added R25: 10K, Resistor_THT:R_Axial_DIN0207_L6.3mm_D2.5mm_P7.62mm_Horizontal, F.Cu at (144.8, 130.2)
- added R26: 1K, Resistor_THT:R_Axial_DIN0207_L6.3mm_D2.5mm_P7.62mm_Horizontal, F.Cu at (144.8, 109.9)
- added R27: 1K, Resistor_THT:R_Axial_DIN0207_L6.3mm_D2.5mm_P7.62mm_Horizontal, F.Cu at (144.8, 122.6)
- added R28: 1K, Resistor_THT:R_Axial_DIN0207_L6.3mm_D2.5mm_P7.62mm_Horizontal, F.Cu at (144.8, 134.0)
- added R29: 10K, Resistor_THT:R_Axial_DIN0207_L6.3mm_D2.5mm_P7.62mm_Horizontal, F.Cu at (182.9, 53.3)
- added R3: 66R, Resistor_THT:R_Axial_DIN0207_L6.3mm_D2.5mm_P7.62mm_Horizontal, F.Cu at (85.1, 94.0)
- added R30: 10K, Resistor_THT:R_Axial_DIN0207_L6.3mm_D2.5mm_P7.62mm_Horizontal, F.Cu at (182.9, 83.8)
- added R31: 10K, Resistor_THT:R_Axial_DIN0207_L6.3mm_D2.5mm_P7.62mm_Horizontal, F.Cu at (182.9, 68.6)
- added R32: 1K, Resistor_THT:R_Axial_DIN0207_L6.3mm_D2.5mm_P7.62mm_Horizontal, F.Cu at (182.9, 58.4)
- added R33: 1K, Resistor_THT:R_Axial_DIN0207_L6.3mm_D2.5mm_P7.62mm_Horizontal, F.Cu at (182.9, 88.9)
- added R34: 1K, Resistor_THT:R_Axial_DIN0207_L6.3mm_D2.5mm_P7.62mm_Horizontal, F.Cu at (190.5, 73.7)
- added R4: 66R, Resistor_THT:R_Axial_DIN0207_L6.3mm_D2.5mm_P7.62mm_Horizontal, F.Cu at (92.1, 94.0)
- added R5: 66R, Resistor_THT:R_Axial_DIN0207_L6.3mm_D2.5mm_P7.62mm_Horizontal, F.Cu at (99.1, 94.0)
- added R6: 66R, Resistor_THT:R_Axial_DIN0207_L6.3mm_D2.5mm_P7.62mm_Horizontal, F.Cu at (106.0, 94.0)
- added R7: 66R, Resistor_THT:R_Axial_DIN0207_L6.3mm_D2.5mm_P7.62mm_Horizontal, F.Cu at (113.0, 94.0)
- added R8: 66R, Resistor_THT:R_Axial_DIN0207_L6.3mm_D2.5mm_P7.62mm_Horizontal, F.Cu at (120.0, 94.0)
- added R9: 1K, Resistor_THT:R_Axial_DIN0207_L6.3mm_D2.5mm_P7.62mm_Horizontal, F.Cu at (120.0, 118.1)
- added U1: 74HC595, Package_DIP:DIP-16_W7.62mm, F.Cu at (104.8, 127.0)
- added U2: 74HC595, Package_DIP:DIP-16_W7.62mm, F.Cu at (157.5, 48.3)
- added U3: 74HC595, Package_DIP:DIP-16_W7.62mm, F.Cu at (157.5, 73.7)
Routing:
- added copper zone on B.Cu, net GND
Other:
- board outline added: 137.2 x 99.1 mm
