File: kicad/small_led_board/small_led_board.kicad_sch (KiCad schematic)
At the start: 107 parts, among them J1 TO FPGA, J2 +5V IN, Q1 IRLZ44N, Q10 IRF4905, Q11 IRF4905, Q12 IRF4905, Q13 IRF4905, Q14 IRF4905, Q15 IRLZ44N, Q16 IRLZ44N, Q17 IRLZ44N, Q18 IRLZ44N, Q19 IRLZ44N, Q2 IRLZ44N, Q20 IRLZ44N, Q3 IRLZ44N, Q4 IRLZ44N, Q5 IRLZ44N, Q6 IRLZ44N, Q7 IRLZ44N, Q8 IRLZ44N, Q9 IRF4905, U1 74HC595, U2 74HC595, U3 74HC595

Commit message: kicad: updated resistor values to 1K
The small led board was barely managing to charge up the shift registers' lines with 10K without any additional strobing.
Now with this change in place, they can strobe four times easily. This is still not nearly the target we want to reach, but it's a first improvement.
Parts:
- R23, R24, R25, R29, R30, R31: value 10K -> 1K
Changed lines of the file:
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@@
       (effects (font (size 1.27 1.27)))
     )
-    (property "Value" "10K" (at 213.36 105.41 90)
+    (property "Value" "1K" (at 213.36 105.41 90)
       (effects (font (size 1.27 1.27)))
     )
@@
       (effects (font (size 1.27 1.27)))
     )
-    (property "Value" "10K" (at 154.94 123.19 90)
+    (property "Value" "1K" (at 154.94 123.19 90)
       (effects (font (size 1.27 1.27)))
     )
@@
       (effects (font (size 1.27 1.27)))
     )
-    (property "Value" "10K" (at 142.24 123.19 90)
+    (property "Value" "1K" (at 142.24 123.19 90)
       (effects (font (size 1.27 1.27)))
     )
@@
       (effects (font (size 1.27 1.27)))
     )
-    (property "Value" "10K" (at 226.06 105.41 90)
+    (property "Value" "1K" (at 226.06 105.41 90)
       (effects (font (size 1.27 1.27)))
     )
@@
       (effects (font (size 1.27 1.27)))
     )
-    (property "Value" "10K" (at 167.64 123.19 90)
+    (property "Value" "1K" (at 167.64 123.19 90)
       (effects (font (size 1.27 1.27)))
     )
@@
       (effects (font (size 1.27 1.27)))
     )
-    (property "Value" "10K" (at 238.76 105.41 90)
-      (effects (font (size 1.27 1.27)))
-    )
+    (property "Value" "1K" (at 238.76 105.41 90)
+      (effects (font (size 1.27 1.27)))
+    )
