File: kicad/small_led_board_v2/small_led_board_v2.kicad_pcb (KiCad board)
At the start: 2 copper layers, 0 parts

Commit message: small led board v2: imported constraints and parts from schematic
Parts:
- added C1: 100nF, Capacitor_THT:C_Disc_D4.7mm_W2.5mm_P5.00mm, F.Cu at (90.0, 105.3)
- added C2: 100nF, Capacitor_THT:C_Disc_D4.7mm_W2.5mm_P5.00mm, F.Cu at (90.0, 109.3)
- added C3: 100nF, Capacitor_THT:C_Disc_D4.7mm_W2.5mm_P5.00mm, F.Cu at (90.0, 113.4)
- added D1: ~, LED_THT:LED_D5.0mm, F.Cu at (61.6, 46.6)
- added D10: ~, LED_THT:LED_D5.0mm, F.Cu at (84.1, 54.2)
- added D11: ~, LED_THT:LED_D5.0mm, F.Cu at (91.6, 54.2)
- added D12: ~, LED_THT:LED_D5.0mm, F.Cu at (99.1, 54.2)
- added D13: ~, LED_THT:LED_D5.0mm, F.Cu at (61.6, 61.7)
- added D14: ~, LED_THT:LED_D5.0mm, F.Cu at (69.1, 61.7)
- added D15: ~, LED_THT:LED_D5.0mm, F.Cu at (76.6, 61.7)
- added D16: ~, LED_THT:LED_D5.0mm, F.Cu at (84.1, 61.7)
- added D17: ~, LED_THT:LED_D5.0mm, F.Cu at (91.6, 61.7)
- added D18: ~, LED_THT:LED_D5.0mm, F.Cu at (99.1, 61.7)
- added D19: ~, LED_THT:LED_D5.0mm, F.Cu at (61.6, 69.3)
- added D2: ~, LED_THT:LED_D5.0mm, F.Cu at (69.1, 46.6)
- added D20: ~, LED_THT:LED_D5.0mm, F.Cu at (69.1, 69.3)
- added D21: ~, LED_THT:LED_D5.0mm, F.Cu at (76.6, 69.3)
- added D22: ~, LED_THT:LED_D5.0mm, F.Cu at (84.1, 69.3)
- added D23: ~, LED_THT:LED_D5.0mm, F.Cu at (91.6, 69.3)
- added D24: ~, LED_THT:LED_D5.0mm, F.Cu at (99.1, 69.3)
- added D25: ~, LED_THT:LED_D5.0mm, F.Cu at (61.6, 76.8)
- added D26: ~, LED_THT:LED_D5.0mm, F.Cu at (69.1, 76.8)
- added D27: ~, LED_THT:LED_D5.0mm, F.Cu at (76.6, 76.8)
- added D28: ~, LED_THT:LED_D5.0mm, F.Cu at (84.1, 76.8)
- added D29: ~, LED_THT:LED_D5.0mm, F.Cu at (91.6, 76.8)
- added D3: ~, LED_THT:LED_D5.0mm, F.Cu at (76.6, 46.6)
- added D30: ~, LED_THT:LED_D5.0mm, F.Cu at (99.1, 76.8)
- added D31: ~, LED_THT:LED_D5.0mm, F.Cu at (61.6, 84.4)
- added D32: ~, LED_THT:LED_D5.0mm, F.Cu at (69.1, 84.4)
- added D33: ~, LED_THT:LED_D5.0mm, F.Cu at (76.6, 84.4)
- added D34: ~, LED_THT:LED_D5.0mm, F.Cu at (84.1, 84.4)
- added D35: ~, LED_THT:LED_D5.0mm, F.Cu at (91.6, 84.4)
- added D36: ~, LED_THT:LED_D5.0mm, F.Cu at (99.1, 84.4)
- added D37: ~, LED_THT:LED_D5.0mm, F.Cu at (61.6, 91.9)
- added D38: ~, LED_THT:LED_D5.0mm, F.Cu at (69.1, 91.9)
- added D39: ~, LED_THT:LED_D5.0mm, F.Cu at (76.6, 91.9)
- added D4: ~, LED_THT:LED_D5.0mm, F.Cu at (84.1, 46.6)
- added D40: ~, LED_THT:LED_D5.0mm, F.Cu at (84.1, 91.9)
- added D41: ~, LED_THT:LED_D5.0mm, F.Cu at (91.6, 91.9)
- added D42: ~, LED_THT:LED_D5.0mm, F.Cu at (99.1, 91.9)
- added D43: ~, LED_THT:LED_D5.0mm, F.Cu at (61.6, 99.5)
- added D44: ~, LED_THT:LED_D5.0mm, F.Cu at (69.1, 99.5)
- added D45: ~, LED_THT:LED_D5.0mm, F.Cu at (76.6, 99.5)
- added D46: ~, LED_THT:LED_D5.0mm, F.Cu at (84.1, 99.5)
- added D47: ~, LED_THT:LED_D5.0mm, F.Cu at (91.6, 99.5)
- added D48: ~, LED_THT:LED_D5.0mm, F.Cu at (99.1, 99.5)
- added D5: ~, LED_THT:LED_D5.0mm, F.Cu at (91.6, 46.6)
- added D6: ~, LED_THT:LED_D5.0mm, F.Cu at (99.1, 46.6)
- added D7: ~, LED_THT:LED_D5.0mm, F.Cu at (61.6, 54.2)
- added D8: ~, LED_THT:LED_D5.0mm, F.Cu at (69.1, 54.2)
- added D9: ~, LED_THT:LED_D5.0mm, F.Cu at (76.6, 54.2)
- added J1: ~, Connector_PinHeader_2.54mm:PinHeader_1x02_P2.54mm_Horizontal, F.Cu at (77.3, 105.6)
- added J2: ~, Connector_BarrelJack:BarrelJack_Horizontal, F.Cu at (123.8, 103.6)
- added J3: ~, Connector_PinSocket_2.54mm:PinSocket_2x05_P2.54mm_Horizontal, F.Cu at (72.7, 105.5)
- added Q1: SQ2351CES, Package_TO_SOT_SMD:SOT-23-3, F.Cu at (106.7, 73.6)
- added Q2: SQ2351CES, Package_TO_SOT_SMD:SOT-23-3, F.Cu at (106.7, 78.2)
- added Q3: SQ2351CES, Package_TO_SOT_SMD:SOT-23-3, F.Cu at (106.7, 82.9)
- added Q4: SQ2351CES, Package_TO_SOT_SMD:SOT-23-3, F.Cu at (106.7, 87.5)
- added Q5: SQ2351CES, Package_TO_SOT_SMD:SOT-23-3, F.Cu at (106.7, 92.1)
- added Q6: SQ2351CES, Package_TO_SOT_SMD:SOT-23-3, F.Cu at (106.7, 96.7)
- added R1: 1M, Resistor_THT:R_Axial_DIN0207_L6.3mm_D2.5mm_P7.62mm_Horizontal, F.Cu at (105.7, 44.9)
- added R10: 150R, Resistor_THT:R_Axial_DIN0207_L6.3mm_D2.5mm_P7.62mm_Horizontal, F.Cu at (116.5, 53.0)
- added R11: 150R, Resistor_THT:R_Axial_DIN0207_L6.3mm_D2.5mm_P7.62mm_Horizontal, F.Cu at (116.5, 57.0)
- added R12: 150R, Resistor_THT:R_Axial_DIN0207_L6.3mm_D2.5mm_P7.62mm_Horizontal, F.Cu at (116.5, 61.1)
- added R13: R, Resistor_THT:R_Axial_DIN0207_L6.3mm_D2.5mm_P7.62mm_Horizontal, F.Cu at (116.5, 65.1)
- added R14: R, Resistor_THT:R_Axial_DIN0207_L6.3mm_D2.5mm_P7.62mm_Horizontal, F.Cu at (116.5, 69.2)
- added R15: R, Resistor_THT:R_Axial_DIN0207_L6.3mm_D2.5mm_P7.62mm_Horizontal, F.Cu at (127.2, 44.9)
- added R16: R, Resistor_THT:R_Axial_DIN0207_L6.3mm_D2.5mm_P7.62mm_Horizontal, F.Cu at (127.2, 48.9)
- added R17: R, Resistor_THT:R_Axial_DIN0207_L6.3mm_D2.5mm_P7.62mm_Horizontal, F.Cu at (127.2, 53.0)
- added R18: R, Resistor_THT:R_Axial_DIN0207_L6.3mm_D2.5mm_P7.62mm_Horizontal, F.Cu at (127.2, 57.0)
- added R19: R, Resistor_THT:R_Axial_DIN0207_L6.3mm_D2.5mm_P7.62mm_Horizontal, F.Cu at (127.2, 61.1)
- added R2: 1M, Resistor_THT:R_Axial_DIN0207_L6.3mm_D2.5mm_P7.62mm_Horizontal, F.Cu at (105.7, 48.9)
- added R20: R, Resistor_THT:R_Axial_DIN0207_L6.3mm_D2.5mm_P7.62mm_Horizontal, F.Cu at (127.2, 65.1)
- added R3: 1M, Resistor_THT:R_Axial_DIN0207_L6.3mm_D2.5mm_P7.62mm_Horizontal, F.Cu at (105.7, 53.0)
- added R4: 1M, Resistor_THT:R_Axial_DIN0207_L6.3mm_D2.5mm_P7.62mm_Horizontal, F.Cu at (105.7, 57.0)
- added R5: 1M, Resistor_THT:R_Axial_DIN0207_L6.3mm_D2.5mm_P7.62mm_Horizontal, F.Cu at (105.7, 61.1)
- added R6: 1M, Resistor_THT:R_Axial_DIN0207_L6.3mm_D2.5mm_P7.62mm_Horizontal, F.Cu at (105.7, 65.1)
- added R7: 150R, Resistor_THT:R_Axial_DIN0207_L6.3mm_D2.5mm_P7.62mm_Horizontal, F.Cu at (105.7, 69.2)
- added R8: 150R, Resistor_THT:R_Axial_DIN0207_L6.3mm_D2.5mm_P7.62mm_Horizontal, F.Cu at (116.5, 44.9)
- added R9: 150R, Resistor_THT:R_Axial_DIN0207_L6.3mm_D2.5mm_P7.62mm_Horizontal, F.Cu at (116.5, 48.9)
- added U1: 74HCT541, Package_DIP:DIP-20_W7.62mm, F.Cu at (110.9, 73.3)
- added U2: 74HCT595, Package_SO:SOIC-16_3.9x9.9mm_P1.27mm, F.Cu at (130.5, 104.1)
- added U3: TPIC6B595N, Package_DIP:DIP-20_W7.62mm, F.Cu at (121.7, 73.3)
Other:
- rule pad_to_mask_clearance: 0 -> 0.038
